File: Lab/Assignment1/Lab_assignment1.kicad_sch (KiCad schematic)
At the start: 35 parts, among them J1 SWD, J2 Conn_01x20, J3 USB_B_Micro, J4 Conn_01x20, SW1 SW_Push, U1 STM32F103C8T6, U2 LM1117I-3.3, U3 HEADER3X2, Y1 8MHZ

Commit message: a2
Parts:
- added D2: 1N4007, Diode_THT:D_DO-41_SOD81_P10.16mm_Horizontal, symbol Diode:1N4007
- added M1: Fan, symbol Motor:Fan
- added Q1: TIP120, Package_TO_SOT_THT:TO-220-3_Vertical, symbol Transistor_BJT:TIP120
- added R11, R12: R, symbol Device:R
- added R13: 1000ohm, symbol Device:R
- added R14, R15: 4.7k ohm, symbol Device:R
- added SW2, SW3, SW4: SW_Push, symbol Switch:SW_Push
- added U4: TC74A0-3.3VAT, TC74A0-3.3VAT:TO170P1054X470X1557-5, symbol TC74A0-3.3VAT:TC74A0-3.3VAT
Connections:
- net GND: now also Q1.3 (E), SW2.2, SW3.2, SW4.2, U4.3 (GND)
- net at J2.19 (Pin_19), U1.11 (PA1): now also R11.2, SW2.1
- new net: D2.2 (A), Q1.1 (B), R13.2
- new net: Q1.2 (C), R12.2
- new net: R14.2, U4.2 (SDA)
- new net: M1.2 (-), R12.1
- new net: R11.1, R13.1
- new net: R15.2, U4.4 (SCLK)
- new net +5V: M1.1 (+), U4.5 (VDD)
- new net PB10: R15.1
- new net PB11: R14.1
